File: kicad/Serial_Breakout.kicad_sch (KiCad schematic)
At the start: 11 parts, among them J10 USB_B_Micro, J9 Serial, U5 FT232RL

Commit message: Rotate Green LED 180 degrees on Serial breakout.
Parts:
- D1R1: LCSC ~C375451 -> C5553577
- D2G1: LCSC ~C375454 -> C6501109
- J10: LCSC ~C598519 -> C3197716
Changed lines of the file:
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@@
       (effects (font (size 1.27 1.27)) hide)
     )
-    (property "LCSC" "~C375451" (id 4) (at 161.29 25.4 0)
+    (property "LCSC" "C5553577" (id 4) (at 161.29 25.4 0)
       (effects (font (size 1.27 1.27)) hide)
     )
@@
       (effects (font (size 1.27 1.27)) hide)
     )
-    (property "LCSC" "~C375454" (id 4) (at 161.29 83.82 0)
+    (property "LCSC" "C6501109" (id 4) (at 161.29 83.82 0)
       (effects (font (size 1.27 1.27)) hide)
     )
@@
       (effects (font (size 1.27 1.27)) hide)
     )
-    (property "LCSC" "~C598519" (id 8) (at 163.83 52.07 0)
-      (effects (font (size 1.27 1.27)) hide)
-    )
+    (property "LCSC" "C3197716" (id 8) (at 163.83 52.07 0)
+      (effects (font (size 1.27 1.27)) hide)
+    )
